File: PCB/kicad_project/mcu.kicad_sch (KiCad schematic)
At the start: 74 parts, among them U1 STM32H750XBHx, U5 IS42S16160J, U6 IS42S16160J, U7 W25Q32JVZP, U8 W25Q32JVZP, Y1 32M, Y2 32.768k

Commit message: 更新物料 删除16bit sdram*2 改为32bit sdram*1
Parts:
- removed R12: 10K, Resistor_SMD:R_0402_1005Metric, symbol Device:R
- removed U5, U6: IS42S16160J, Package_BGA:Alliance_TFBGA-54_8x8mm_Layout9x9_P0.8mm, symbol my:IS42S16160J-6BL
- added U9: ~, Package_BGA:BGA-90_8.0x13.0mm_Layout2x3x15_P0.8mm, symbol my:IS42S32160D
Connections:
- net DGND: now also U9.A3 (VSS), U9.B3 (VSSQ), U9.B8 (VSSQ), U9.C1 (VSSQ), U9.D1 (VSSQ), U9.E9 (VSSQ), U9.F1 (VSS), U9.L3 (VSS), U9.L9 (VSSQ), U9.M1 (VSSQ), U9.N1 (VSSQ), U9.P3 (VSSQ), U9.P8 (VSSQ), U9.R3 (VSS)
- net SDRAM_A0: now also U9.G8 (A0)
- net SDRAM_A1: now also U9.G9 (A1)
- net SDRAM_A10: now also U9.G7 (A10)
- net SDRAM_A11: now also U9.H9 (A11)
- net SDRAM_A12: now also U9.H3 (A12)
- net SDRAM_A2: now also U9.F7 (A2)
- net SDRAM_A3: now also U9.F3 (A3)
- net SDRAM_A4: now also U9.G1 (A4)
- net SDRAM_A5: now also U9.G2 (A5)
- net SDRAM_A6: now also U9.G3 (A6)
- net SDRAM_A7: now also U9.H1 (A7)
- net SDRAM_A8: now also U9.H2 (A8)
- net SDRAM_A9: now also U9.J3 (A9)
- net SDRAM_BA0: now also U9.J7 (BA0)
- net SDRAM_BA1: now also U9.H8 (BA1)
- net SDRAM_CAS: now also U9.K7 (CAS#)
- net SDRAM_CKE: now also U9.J2 (CKE)
- net SDRAM_CLK: now also U9.J1 (CLK)
- net SDRAM_CS#: now also U9.J8 (CS#)
- net SDRAM_D0: now also U9.R8 (DQ0)
- net SDRAM_D1: now also U9.N7 (DQ1)
- net SDRAM_D10: now also U9.M2 (DQ10)
- net SDRAM_D11: now also U9.P1 (DQ11)
- net SDRAM_D12: now also U9.N2 (DQ12)
- net SDRAM_D13: now also U9.R1 (DQ13)
- net SDRAM_D14: now also U9.N3 (DQ14)
- net SDRAM_D15: now also U9.R2 (DQ15)
- net SDRAM_D16: now also U9.E8 (DQ16)
- net SDRAM_D17: now also U9.D7 (DQ17)
- net SDRAM_D18: now also U9.D8 (DQ18)
- net SDRAM_D19: now also U9.B9 (DQ19)
- net SDRAM_D2: now also U9.R9 (DQ2)
- net SDRAM_D20: now also U9.C8 (DQ20)
- net SDRAM_D21: now also U9.A9 (DQ21)
- net SDRAM_D22: now also U9.C7 (DQ22)
- net SDRAM_D23: now also U9.A8 (DQ23)
- net SDRAM_D24: now also U9.A2 (DQ24)
- net SDRAM_D25: now also U9.C3 (DQ25)
- net SDRAM_D26: now also U9.A1 (DQ26)
- net SDRAM_D27: now also U9.C2 (DQ27)
- net SDRAM_D28: now also U9.B1 (DQ28)
- net SDRAM_D29: now also U9.D2 (DQ29)
- net SDRAM_D3: now also U9.N8 (DQ3)
- net SDRAM_D30: now also U9.D3 (DQ30)
- net SDRAM_D31: now also U9.E2 (DQ31)
- net SDRAM_D4: now also U9.P9 (DQ4)
- net SDRAM_D5: now also U9.M8 (DQ5)
- net SDRAM_D6: now also U9.M7 (DQ6)
- net SDRAM_D7: now also U9.L8 (DQ7)
- net SDRAM_D8: now also U9.L2 (DQ8)
- net SDRAM_D9: now also U9.M3 (DQ9)
- net SDRAM_DQM0: now also U9.K9 (DQM0)
- net SDRAM_DQM1: now also U9.K1 (DQM1)
- net SDRAM_DQM2: now also U9.F8 (DQM2)
- net SDRAM_DQM3: now also U9.F2 (DQM3)
- net SDRAM_RAS: now also U9.J9 (RAS#)
- net SDRAM_WE: now also U9.K8 (WE#)
- net VDD: now also C27.1, C28.1, C29.1, U1.F17 (VDD33_USB), U1.G17 (VDD50_USB), U9.A7 (VDD), U9.B2 (VDDQ), U9.B7 (VDDQ), U9.C9 (VDDQ), U9.D9 (VDDQ), U9.E1 (VDDQ), U9.F9 (VDD), U9.L1 (VDDQ), U9.L7 (VDD), U9.M9 (VDDQ), U9.N9 (VDDQ), U9.P2 (VDDQ), U9.P7 (VDDQ), U9.R7 (VDD)
Other:
- moved on the sheet: C63, C64, U7, U8

Commit message: MCU部分扇出，SDRAM走线ing
Other:
- moved on the sheet: R5
Changed lines of the file:
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@@
 	(wire
 		(pts
-			(xy 335.28 214.63) (xy 346.71 214.63)
-		)
-		(stroke
-			(width 0)
-			(type default)
-		)
-	)
-	(wire
-		(pts
 			(xy 198.12 248.92) (xy 209.55 248.92)
 		)
@@
 	(wire
 		(pts
-			(xy 328.93 219.71) (xy 346.71 219.71)
+			(xy 325.12 219.71) (xy 346.71 219.71)
 		)
 		(stroke
@@
 	(wire
 		(pts
-			(xy 335.28 212.09) (xy 346.71 212.09)
+			(xy 334.01 212.09) (xy 346.71 212.09)
 		)
 		(stroke
@@
 	(wire
 		(pts
-			(xy 335.28 227.33) (xy 346.71 227.33)
+			(xy 334.01 227.33) (xy 346.71 227.33)
 		)
 		(stroke
@@
 	(wire
 		(pts
+			(xy 334.01 214.63) (xy 346.71 214.63)
+		)
+		(stroke
+			(width 0)
+			(type default)
+		)
+	)
+	(wire
+		(pts
 			(xy 130.81 39.37) (xy 138.43 39.37)
 		)
@@
 	(wire
 		(pts
-			(xy 335.28 224.79) (xy 346.71 224.79)
+			(xy 334.01 224.79) (xy 346.71 224.79)
 		)
 		(stroke
@@
 	(wire
 		(pts
-			(xy 335.28 222.25) (xy 346.71 222.25)
+			(xy 334.01 222.25) (xy 346.71 222.25)
 		)
 		(stroke
@@
 	(wire
 		(pts
+			(xy 334.01 217.17) (xy 346.71 217.17)
+		)
+		(stroke
+			(width 0)
+			(type default)
+		)
+	)
+	(wire
+		(pts
 			(xy 389.89 262.89) (xy 378.46 262.89)
 		)
@@
 	(wire
 		(pts
-			(xy 335.28 229.87) (xy 346.71 229.87)
+			(xy 334.01 229.87) (xy 346.71 229.87)
 		)
 		(stroke
@@
 	(wire
 		(pts
-			(xy 335.28 217.17) (xy 346.71 217.17)
-		)
-		(stroke
-			(width 0)
-			(type default)
-		)
-	)
-	(wire
-		(pts
 			(xy 87.63 152.4) (xy 99.06 152.4)
 		)
@@
 	(hierarchical_label "VDD"
 		(shape input)
-		(at 321.31 219.71 180)
+		(at 317.5 219.71 180)
 		(fields_autoplaced yes)
 		(effects
@@
 		(length 2.54)
 		(shape round)
+		(at 334.01 222.25 0)
+		(fields_autoplaced yes)
+		(effects
+			(font
+				(size 1.27 1.27)
+			)
+			(justify left bottom)
+		)
+		(property "Netclass" "sdram_ctrl"
+			(at 333.3115 219.71 0)
+			(effects
+				(font
+					(size 1.27 1.27)
+					(italic yes)
+				)
+				(justify right)
+			)
+		)
+	)
+	(netclass_flag ""
+		(length 2.54)
+		(shape round)
+		(at 334.01 212.09 0)
+		(fields_autoplaced yes)
+		(effects
+			(font
+				(size 1.27 1.27)
+			)
+			(justify left bottom)
+		)
+		(property "Netclass" "sdram_ctrl"
+			(at 333.3115 209.55 0)
+			(effects
+				(font
+					(size 1.27 1.27)
+					(italic yes)
+				)
+				(justify right)
+			)
+		)
+	)
+	(netclass_flag ""
+		(length 2.54)
+		(shape round)
+		(at 334.01 227.33 0)
+		(fields_autoplaced yes)
+		(effects
+			(font
+				(size 1.27 1.27)
+			)
+			(justify left bottom)
+		)
+		(property "Netclass" "sdram_ctrl"
+			(at 333.3115 224.79 0)
+			(effects
+				(font
+					(size 1.27 1.27)
+					(italic yes)
+				)
+				(justify right)
+			)
+		)
+	)
+	(netclass_flag ""
+		(length 2.54)
+		(shape round)
+		(at 334.01 229.87 0)
+		(fields_autoplaced yes)
+		(effects
+			(font
+				(size 1.27 1.27)
+			)
+			(justify left bottom)
+		)
+		(property "Netclass" "sdram_ctrl"
+			(at 333.3115 227.33 0)
+			(effects
+				(font
+					(size 1.27 1.27)
+					(italic yes)
+				)
+				(justify right)
+			)
+		)
+	)
+	(netclass_flag ""
+		(length 2.54)
+		(shape round)
+		(at 334.01 214.63 0)
+		(fields_autoplaced yes)
+		(effects
+			(font
+				(size 1.27 1.27)
+			)
+			(justify left bottom)
+		)
+		(property "Netclass" "sdram_ctrl"
+			(at 333.3115 212.09 0)
+			(effects
+				(font
+					(size 1.27 1.27)
+					(italic yes)
+				)
+				(justify right)
+			)
+		)
+	)
+	(netclass_flag ""
+		(length 2.54)
+		(shape round)
+		(at 334.01 224.79 0)
+		(fields_autoplaced yes)
+		(effects
+			(font
+				(size 1.27 1.27)
+			)
+			(justify left bottom)
+		)
+		(property "Netclass" "sdram_ctrl"
+			(at 333.3115 222.25 0)
+			(effects
+				(font
+					(size 1.27 1.27)
+					(italic yes)
+				)
+				(justify right)
+			)
+		)
+	)
+	(netclass_flag ""
+		(length 2.54)
+		(shape round)
 		(at 181.61 39.37 0)
 		(fields_autoplaced yes)
@@
 		)
 	)
+	(netclass_flag ""
+		(length 2.54)
+		(shape round)
+		(at 334.01 219.71 0)
+		(fields_autoplaced yes)
+		(effects
+			(font
+				(size 1.27 1.27)
+			)
+			(justify left bottom)
+		)
+		(property "Netclass" "sdram_ctrl"
+			(at 333.3115 217.17 0)
+			(effects
+				(font
+					(size 1.27 1.27)
+					(italic yes)
+				)
+				(justify right)
+			)
+		)
+	)
+	(netclass_flag ""
+		(length 2.54)
+		(shape round)
+		(at 334.01 217.17 0)
+		(fields_autoplaced yes)
+		(effects
+			(font
+				(size 1.27 1.27)
+			)
+			(justify left bottom)
+		)
+		(property "Netclass" "sdram_ctrl"
+			(at 333.3115 214.63 0)
+			(effects
+				(font
+					(size 1.27 1.27)
+					(italic yes)
+				)
+				(justify right)
+			)
+		)
+	)
 	(symbol
 		(lib_id "Device:C")
@@
 	(symbol
 		(lib_id "Device:R")
-		(at 325.12 219.71 90)
+		(at 321.31 219.71 90)
 		(unit 1)
 		(exclude_from_sim no)
@@
 		(dnp no)
 		(property "Reference" "R5"
-			(at 325.12 217.678 90)
+			(at 321.31 217.678 90)
 			(effects
 				(font
@@
 		)
 		(property "Value" "10K"
-			(at 325.12 219.71 90)
+			(at 321.31 219.71 90)
 			(effects
 				(font
@@
 		)
 		(property "Footprint" "Resistor_SMD:R_0402_1005Metric"
-			(at 325.12 221.488 90)
+			(at 321.31 221.488 90)
 			(effects
 				(font
@@
 		)
 		(property "Datasheet" "~"
-			(at 325.12 219.71 0)
+			(at 321.31 219.71 0)
 			(effects
 				(font
@@
 		)
 		(property "Description" "Resistor"
-			(at 325.12 219.71 0)
+			(at 321.31 219.71 0)
 			(effects
 				(font

Commit message: 绕走SDRAM走线。。因复杂度太高，放弃做等长 目前差最后几根数据线，可视情况交换线序
Connections:
- net SDRAM_D19: now also U9.C8 (DQ20); no longer U9.B9 (DQ19)
- net SDRAM_D20: now also U9.C7 (DQ22); no longer U9.C8 (DQ20)
- net SDRAM_D21: now also U9.A8 (DQ23); no longer U9.A9 (DQ21)
- net SDRAM_D22: now also U9.B9 (DQ19); no longer U9.C7 (DQ22)
- net SDRAM_D23: now also U9.A9 (DQ21); no longer U9.A8 (DQ23)
- net SDRAM_D25: now also U9.B1 (DQ28); no longer U9.C3 (DQ25)
- net SDRAM_D26: now also U9.C2 (DQ27); no longer U9.A1 (DQ26)
- net SDRAM_D27: now also U9.A1 (DQ26); no longer U9.C2 (DQ27)
- net SDRAM_D28: now also U9.E2 (DQ31); no longer U9.B1 (DQ28)
- net SDRAM_D29: now also U9.C3 (DQ25); no longer U9.D2 (DQ29)
- net SDRAM_D31: now also U9.D2 (DQ29); no longer U9.E2 (DQ31)
Changed lines of the file:
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@@
-		)
-	)
-	(label "SDRAM_D22"
-		(at 389.89 242.57 180)
-		(fields_autoplaced yes)
-		(effects
-			(font
-				(size 1.27 1.27)
-			)
-			(justify right bottom)
 		)
 	)
@@
 		)
 	)
+	(label "SDRAM_D26"
+		(at 389.89 260.35 180)
+		(fields_autoplaced yes)
+		(effects
+			(font
+				(size 1.27 1.27)
+			)
+			(justify right bottom)
+		)
+	)
 	(label "QSPI2_IO3"
 		(at 87.63 271.78 0)
@@
 		)
 	)
+	(label "SDRAM_D21"
+		(at 389.89 245.11 180)
+		(fields_autoplaced yes)
+		(effects
+			(font
+				(size 1.27 1.27)
+			)
+			(justify right bottom)
+		)
+	)
 	(label "SDRAM_D31"
 		(at 87.63 175.26 0)
@@
 		)
 	)
+	(label "SDRAM_D19"
+		(at 389.89 237.49 180)
+		(fields_autoplaced yes)
+		(effects
+			(font
+				(size 1.27 1.27)
+			)
+			(justify right bottom)
+		)
+	)
 	(label "SDRAM_D15"
 		(at 198.12 228.6 0)
@@
 		)
 	)
+	(label "SDRAM_D31"
+		(at 389.89 265.43 180)
+		(fields_autoplaced yes)
+		(effects
+			(font
+				(size 1.27 1.27)
+			)
+			(justify right bottom)
+		)
+	)
 	(label "QSPI_CS"
 		(at 334.01 336.55 0)
@@
 		)
 	)
-	(label "SDRAM_D27"
-		(at 389.89 260.35 180)
-		(fields_autoplaced yes)
-		(effects
-			(font
-				(size 1.27 1.27)
-			)
-			(justify right bottom)
-		)
-	)
 	(label "SDRAM_D24"
 		(at 389.89 252.73 180)
@@
 		)
 	)
+	(label "SDRAM_D28"
+		(at 389.89 270.51 180)
+		(fields_autoplaced yes)
+		(effects
+			(font
+				(size 1.27 1.27)
+			)
+			(justify right bottom)
+		)
+	)
 	(label "SDRAM_D12"
 		(at 389.89 212.09 180)
@@
 		)
 	)
-	(label "SDRAM_D20"
-		(at 389.89 237.49 180)
-		(fields_autoplaced yes)
-		(effects
-			(font
-				(size 1.27 1.27)
-			)
-			(justify right bottom)
-		)
-	)
 	(label "SDRAM_D13"
 		(at 198.12 223.52 0)
@@
 		)
 	)
+	(label "SDRAM_D20"
+		(at 389.89 242.57 180)
+		(fields_autoplaced yes)
+		(effects
+			(font
+				(size 1.27 1.27)
+			)
+			(justify right bottom)
+		)
+	)
 	(label "SDRAM_A3"
 		(at 334.01 181.61 0)
@@
 		)
 	)
-	(label "SDRAM_D19"
-		(at 389.89 234.95 180)
-		(fields_autoplaced yes)
-		(effects
-			(font
-				(size 1.27 1.27)
-			)
-			(justify right bottom)
-		)
-	)
 	(label "QSPI1_IO2"
 		(at 209.55 251.46 180)
@@
 		)
 	)
-	(label "SDRAM_D29"
-		(at 389.89 265.43 180)
-		(fields_autoplaced yes)
-		(effects
-			(font
-				(size 1.27 1.27)
-			)
-			(justify right bottom)
-		)
-	)
 	(label "SDRAM_CKE"
 		(at 335.28 222.25 0)
@@
 		)
 	)
+	(label "SDRAM_D25"
+		(at 389.89 262.89 180)
+		(fields_autoplaced yes)
+		(effects
+			(font
+				(size 1.27 1.27)
+			)
+			(justify right bottom)
+		)
+	)
 	(label "SDRAM_D2"
 		(at 389.89 181.61 180)
@@
 		)
 	)
-	(label "SDRAM_D21"
-		(at 389.89 240.03 180)
-		(fields_autoplaced yes)
-		(effects
-			(font
-				(size 1.27 1.27)
-			)
-			(justify right bottom)
-		)
-	)
 	(label "SDRAM_CS#"
 		(at 198.12 160.02 0)
@@
 		)
 	)
-	(label "SDRAM_D31"
-		(at 389.89 270.51 180)
-		(fields_autoplaced yes)
-		(effects
-			(font
-				(size 1.27 1.27)
-			)
-			(justify right bottom)
-		)
-	)
 	(label "QSPI1_IO0"
 		(at 284.48 341.63 0)
@@
 		)
 	)
+	(label "SDRAM_D27"
+		(at 389.89 257.81 180)
+		(fields_autoplaced yes)
+		(effects
+			(font
+				(size 1.27 1.27)
+			)
+			(justify right bottom)
+		)
+	)
 	(label "SDRAM_D8"
 		(at 198.12 274.32 0)
@@
 		)
 	)
-	(label "SDRAM_D26"
-		(at 389.89 257.81 180)
-		(fields_autoplaced yes)
-		(effects
-			(font
-				(size 1.27 1.27)
-			)
-			(justify right bottom)
-		)
-	)
 	(label "QSPI_CS"
 		(at 209.55 187.96 180)
@@
 		)
 	)
+	(label "SDRAM_D29"
+		(at 389.89 255.27 180)
+		(fields_autoplaced yes)
+		(effects
+			(font
+				(size 1.27 1.27)
+			)
+			(justify right bottom)
+		)
+	)
 	(label "SDRAM_DQM1"
 		(at 198.12 248.92 0)
@@
 		)
 	)
+	(label "SDRAM_D23"
+		(at 389.89 240.03 180)
+		(fields_autoplaced yes)
+		(effects
+			(font
+				(size 1.27 1.27)
+			)
+			(justify right bottom)
+		)
+	)
 	(label "SDRAM_DQM1"
 		(at 392.43 199.39 180)
@@
 		)
 	)
-	(label "SDRAM_D28"
-		(at 389.89 262.89 180)
-		(fields_autoplaced yes)
-		(effects
-			(font
-				(size 1.27 1.27)
-			)
-			(justify right bottom)
-		)
-	)
 	(label "SDRAM_D30"
 		(at 389.89 267.97 180)
@@
 		)
 	)
-	(label "SDRAM_D23"
-		(at 389.89 245.11 180)
-		(fields_autoplaced yes)
-		(effects
-			(font
-				(size 1.27 1.27)
-			)
-			(justify right bottom)
-		)
-	)
 	(label "QSPI_CS"
 		(at 284.48 336.55 0)
@@
 		)
 	)
-	(label "SDRAM_D25"
-		(at 389.89 255.27 180)
-		(fields_autoplaced yes)
-		(effects
+	(label "SDRAM_D22"
+		(at 389.89 234.95 180)
+		(fields_autoplaced yes)
+		(effects

Commit message: 完成了SDRAM和QSPI的走线，QSPI做了网络等长匹配（两根复用线未连接以用于准确计算线长）
Connections:
- net SDRAM_D12: now also U9.L2 (DQ8); no longer U9.N2 (DQ12)
- net SDRAM_D8: now also U9.N2 (DQ12); no longer U9.L2 (DQ8)
- net USB_FS_D+: now reaches U1.E16 (PA12)
- net USB_FS_D-: now reaches U1.E17 (PA11)
Changed lines of the file:
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@@
 	(wire
 		(pts
+			(xy 198.12 99.06) (xy 201.93 99.06)
+		)
+		(stroke
+			(width 0)
+			(type default)
+		)
+	)
+	(wire
+		(pts
 			(xy 116.84 33.02) (xy 124.46 33.02)
 		)
@@
 	(wire
 		(pts
+			(xy 198.12 96.52) (xy 201.93 96.52)
+		)
+		(stroke
+			(width 0)
+			(type default)
+		)
+	)
+	(wire
+		(pts
 			(xy 374.65 130.81) (xy 374.65 133.35)
 		)
@@
 		)
 	)
-	(label "SDRAM_D12"
-		(at 389.89 212.09 180)
-		(fields_autoplaced yes)
-		(effects
-			(font
-				(size 1.27 1.27)
-			)
-			(justify right bottom)
-		)
-	)
 	(label "VDDA"
 		(at 175.26 39.37 0)
@@
 		)
 	)
+	(label "SDRAM_D8"
+		(at 389.89 212.09 180)
+		(fields_autoplaced yes)
+		(effects
+			(font
+				(size 1.27 1.27)
+			)
+			(justify right bottom)
+		)
+	)
 	(label "SDRAM_D9"
 		(at 198.12 276.86 0)
@@
 		)
 	)
-	(label "SDRAM_D8"
-		(at 389.89 201.93 180)
-		(fields_autoplaced yes)
-		(effects
-			(font
-				(size 1.27 1.27)
-			)
-			(justify right bottom)
-		)
-	)
 	(label "SDRAM_WE"
 		(at 87.63 205.74 0)
@@
 		)
 	)
+	(label "SDRAM_D12"
+		(at 389.89 201.93 180)
+		(fields_autoplaced yes)
+		(effects
+			(font
+				(size 1.27 1.27)
+			)
+			(justify right bottom)
+		)
+	)
 	(label "SDRAM_CKE"
 		(at 198.12 165.1 0)
@@
 		)
 	)
+	(hierarchical_label "USB_FS_D-"
+		(shape bidirectional)
+		(at 201.93 96.52 0)
+		(fields_autoplaced yes)
+		(effects
+			(font
+				(size 1.27 1.27)
+			)
+			(justify left)
+		)
+	)
+	(hierarchical_label "USB_FS_D+"
+		(shape bidirectional)
+		(at 201.93 99.06 0)
+		(fields_autoplaced yes)
+		(effects
+			(font
+				(size 1.27 1.27)
+			)
+			(justify left)
+		)
+	)
 	(hierarchical_label "DGND"
 		(shape input)
@@
 		)
 		(pin "E17"
+			(alternate "USB_OTG_FS_DM")
 		)
 		(pin "E8"
@@
 		)
 		(pin "E16"
+			(alternate "USB_OTG_FS_DP")
 		)
 		(pin "E10"

Commit message: 铺铜，增加BTB
Parts:
- C16, C2: footprint Capacitor_SMD:C_0201_0603Metric_Pad0.64x0.40mm_HandSolder -> Capacitor_SMD:C_0402_1005Metric
Connections:
- net USB_FS_D+: no longer names the net of U1.E16 (PA12)
- net USB_FS_D-: no longer names the net of U1.E17 (PA11)
Changed lines of the file:
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@@
 	(wire
 		(pts
-			(xy 198.12 99.06) (xy 201.93 99.06)
-		)
-		(stroke
-			(width 0)
-			(type default)
-		)
-	)
-	(wire
-		(pts
 			(xy 116.84 33.02) (xy 124.46 33.02)
 		)
@@
 	(wire
 		(pts
-			(xy 198.12 96.52) (xy 201.93 96.52)
-		)
-		(stroke
-			(width 0)
-			(type default)
-		)
-	)
-	(wire
-		(pts
 			(xy 374.65 130.81) (xy 374.65 133.35)
 		)
@@
 		)
 	)
-	(hierarchical_label "USB_FS_D-"
-		(shape bidirectional)
-		(at 201.93 96.52 0)
-		(fields_autoplaced yes)
-		(effects
-			(font
-				(size 1.27 1.27)
-			)
-			(justify left)
-		)
-	)
-	(hierarchical_label "USB_FS_D+"
-		(shape bidirectional)
-		(at 201.93 99.06 0)
-		(fields_autoplaced yes)
-		(effects
-			(font
-				(size 1.27 1.27)
-			)
-			(justify left)
-		)
-	)
 	(hierarchical_label "DGND"
 		(shape input)
@@
 			)
 		)
-		(property "Footprint" "Capacitor_SMD:C_0201_0603Metric_Pad0.64x0.40mm_HandSolder"
+		(property "Footprint" "Capacitor_SMD:C_0402_1005Metric"
 			(at 224.4852 33.02 0)
 			(effects
@@
 		)
 		(instances
-			(project ""
+			(project "h750xb_core"
 				(path "/a69f31b1-c3a2-49f5-a533-af75e45f29ed/7c8a82fa-473c-4565-a293-03fd63e136b1"
 					(reference "U9")
@@
 		)
 		(pin "E17"
-			(alternate "USB_OTG_FS_DM")
+			(alternate "PA11")
 		)
 		(pin "E8"
@@
 		)
 		(pin "E16"
-			(alternate "USB_OTG_FS_DP")
+			(alternate "PA12")
 		)
 		(pin "E10"
@@
 			)
 		)
-		(property "Footprint" "Capacitor_SMD:C_0201_0603Metric_Pad0.64x0.40mm_HandSolder"
+		(property "Footprint" "Capacitor_SMD:C_0402_1005Metric"
 			(at 117.8052 33.02 0)
 			(effects
@@
 		)
 		(instances
-			(project ""
+			(project "h750xb_core"
 				(path "/a69f31b1-c3a2-49f5-a533-af75e45f29ed/7c8a82fa-473c-4565-a293-03fd63e136b1"
 					(reference "U9")
