File: PCB/kicad_project/mcu.kicad_sch (KiCad schematic)
At the start: 72 parts, among them U1 STM32H750XBHx, U7 W25Q32JVZP, U8 W25Q32JVZP, Y1 32M, Y2 32.768k

Commit message: 收尾
Parts:
- added J1, J2: DF40C-100DP-0.4V_51_, HRS:HIROSE_DF40C-100DP-0.4V_51_, symbol DF40C-100DP-0.4V_51_:DF40C-100DP-0.4V_51_

Commit message: 更新原理图网络和PCB部分IO走线
Parts:
- removed J1, J2: DF40C-100DP-0.4V_51_, HRS:HIROSE_DF40C-100DP-0.4V_51_, symbol DF40C-100DP-0.4V_51_:DF40C-100DP-0.4V_51_
Connections:
- net PD5: now reaches U1.A11 (PD5)
- net PD4: now reaches U1.A12 (PD4)
- net PA15: now reaches U1.A14 (PA15)
- net PB5: now reaches U1.A5 (PB5)
- net PK5: now reaches U1.A8 (PK5)
- net PG10: now reaches U1.A9 (PG10)
- net PJ15: now reaches U1.B10 (PJ15)
- net PD6: now reaches U1.B11 (PD6)
- net PD3: now reaches U1.B12 (PD3)
- net PA14: now reaches U1.B14 (PA14)
- net PB6: now reaches U1.B5 (PB6)
- net PB4: now reaches U1.B7 (PB4)
- net PK4: now reaches U1.B8 (PK4)
- net PG11: now reaches U1.B9 (PG11)
- net PD7: now reaches U1.C11 (PD7)
- net PC12: now reaches U1.C12 (PC12)
- net PA13: now reaches U1.C15 (PA13)
- net PB7: now reaches U1.C5 (PB7)
- net PB3: now reaches U1.C6 (PB3)
- net PK6: now reaches U1.C7 (PK6)
- net PK3: now reaches U1.C8 (PK3)
- net PG12: now reaches U1.C9 (PG12)
- net PE5: now reaches U1.D1 (PE5)
- net PJ14: now reaches U1.D10 (PJ14)
- net PJ12: now reaches U1.D11 (PJ12)
- net PD2: now reaches U1.D12 (PD2)
- net PA10: now reaches U1.D14 (PA10)
- net PA9: now reaches U1.D15 (PA9)
- net PE4: now reaches U1.D2 (PE4)
- net PE3: now reaches U1.D3 (PE3)
- net PB9: now reaches U1.D4 (PB9)
- net PB8: now reaches U1.D5 (PB8)
- net PK7: now reaches U1.D7 (PK7)
- net PG13: now reaches U1.D9 (PG13)
- net PJ13: now reaches U1.E10 (PJ13)
- net PC8: now reaches U1.E13 (PC8)
- net PA8: now reaches U1.E15 (PA8)
- net PA12: now reaches U1.E16 (PA12)
- net PA11: now reaches U1.E17 (PA11)
- net PC13: now reaches U1.E3 (PC13)
- net PI8: now reaches U1.E4 (PI8)
- net PE6: now reaches U1.E5 (PE6)
- net PC7: now reaches U1.F13 (PC7)
- net PC6: now reaches U1.F14 (PC6)
- net PG7: now reaches U1.F16 (PG7)
- net PI11: now reaches U1.F4 (PI11)
- net PG6: now reaches U1.G15 (PG6)
- net PI12: now reaches U1.H1 (PI12)
- net PG3: now reaches U1.H15 (PG3)
- net PK2: now reaches U1.H17 (PK2)
- net PI13: now reaches U1.H2 (PI13)
- net PI14: now reaches U1.H3 (PI14)
- net PK0: now reaches U1.J14 (PK0)
- net PK1: now reaches U1.J15 (PK1)
- net PJ11: now reaches U1.K14 (PJ11)
- net PF7: now reaches U1.K3 (PF7)
- net PF8: now reaches U1.K4 (PF8)
- net PJ10: now reaches U1.L14 (PJ10)
- net PC0: now reaches U1.L2 (PC0)
- net PF9: now reaches U1.L4 (PF9)
- net PJ9: now reaches U1.M14 (PJ9)
- net PC1: now reaches U1.M2 (PC1)
- net PJ8: now reaches U1.N13 (PJ8)
- net PJ7: now reaches U1.N14 (PJ7)
- net PJ6: now reaches U1.N15 (PJ6)
- net PA2: now reaches U1.N3 (PA2)
- net PA1: now reaches U1.N4 (PA1)
- net PA0: now reaches U1.N5 (PA0)
- net PJ0: now reaches U1.N6 (PJ0)
- net PB10: now reaches U1.P11 (PB10)
- net PB11: now reaches U1.P12 (PB11)
- net PH4: now reaches U1.P3 (PH4)
- net PI15: now reaches U1.P5 (PI15)
- net PJ1: now reaches U1.P6 (PJ1)
- net PC2_C: now reaches U1.R1 (PC2_C)
- net PJ5: now reaches U1.R12 (PJ5)
- net PD11: now reaches U1.R15 (PD11)
- net PD12: now reaches U1.R16 (PD12)
- net PD13: now reaches U1.R17 (PD13)
- net PC3_C: now reaches U1.R2 (PC3_C)
- net PA6: now reaches U1.R3 (PA6)
- net PA7: now reaches U1.R5 (PA7)
- net PB2: now reaches U1.R6 (PB2)
- net PA0_C: now reaches U1.T1 (PA0_C)
- net PH6: now reaches U1.T11 (PH6)
- net PB12: now reaches U1.T14 (PB12)
- net PB15: now reaches U1.T15 (PB15)
- net PA1_C: now reaches U1.T2 (PA1_C)
- net PA5: now reaches U1.T3 (PA5)
- net PC4: now reaches U1.T4 (PC4)
- net PB1: now reaches U1.T5 (PB1)
- net PJ2: now reaches U1.T6 (PJ2)
- net PH7: now reaches U1.U13 (PH7)
- net PB13: now reaches U1.U14 (PB13)
- net PB14: now reaches U1.U15 (PB14)
- net PA3: now reaches U1.U2 (PA3)
- net PA4: now reaches U1.U3 (PA4)
- net PC5: now reaches U1.U4 (PC5)
- net PB0: now reaches U1.U5 (PB0)
- net PJ3: now reaches U1.U6 (PJ3)
- net PJ4: now reaches U1.U7 (PJ4)
Other:
- moved on the sheet: C65, C66, C67, C68, Y1, Y2
