File: PCB/kicad_project/h750xb_core.kicad_pcb (KiCad board)
At the start: 6 copper layers, 50 x 35 mm, 93 parts, among them J1 DF40C-100DP-0.4V_51_, J2 DF40C-100DP-0.4V_51_, U1 STM32H750XBHx, U2 TPS74801DRC, U3 TPS82130, U4 REF3020, U7 W25Q32JVZP, U8 W25Q32JVZP, Y1 32M, Y2 32.768k

Commit message: 完工0-0
Parts:
- moved R4 1.02 mm to (25.9, 81.0)
- moved R11 0.80 mm to (25.1, 80.2), turned to 90 degrees
Connections:
- net /mcu/PI11 renamed /PI11
- net /mcu/PI12 renamed /PI12
- net /mcu/PI13 renamed /PI13
- net /mcu/PI14 renamed /PI14
- net /mcu/PI15 renamed /PI15
- net /mcu/PI8 renamed /PI8
- net /mcu/PJ0 renamed /PJ0
- net /mcu/PJ1 renamed /PJ1
- net /mcu/PJ13 renamed /PJ13
- net /mcu/PJ14 renamed /PJ14
- net /mcu/PJ2 renamed /PJ2
- net /mcu/PJ3 renamed /PJ3
- net /mcu/PJ4 renamed /PJ4
- net /mcu/PK6 renamed /PK6
- net /mcu/PK7 renamed /PK7
- D3 pad 1: /ex_VBAT -> GND
- J1 pad 1: unconnected-(J1-Pad1) -> GND
- J1 pad 10: unconnected-(J1-Pad10) -> /PD2
- J1 pad 100: unconnected-(J1-Pad100) -> GND
- J1 pad 11: unconnected-(J1-Pad11) -> /PG11
- J1 pad 12: unconnected-(J1-Pad12) -> GND
- J1 pad 13: unconnected-(J1-Pad13) -> GND
- J1 pad 14: unconnected-(J1-Pad14) -> /PA13
- J1 pad 15: unconnected-(J1-Pad15) -> /PJ15
- J1 pad 16: unconnected-(J1-Pad16) -> GND
- J1 pad 17: unconnected-(J1-Pad17) -> GND
- J1 pad 18: unconnected-(J1-Pad18) -> /PA12
- J1 pad 19: unconnected-(J1-Pad19) -> /PD7
- J1 pad 2: unconnected-(J1-Pad2) -> GND
- J1 pad 20: unconnected-(J1-Pad20) -> /PA11
- J1 pad 21: unconnected-(J1-Pad21) -> GND
- J1 pad 22: unconnected-(J1-Pad22) -> GND
- J1 pad 23: unconnected-(J1-Pad23) -> /PD6
- J1 pad 24: unconnected-(J1-Pad24) -> /PA10
- J1 pad 25: unconnected-(J1-Pad25) -> GND
- J1 pad 26: unconnected-(J1-Pad26) -> GND
- J1 pad 27: unconnected-(J1-Pad27) -> /PD5
- J1 pad 28: unconnected-(J1-Pad28) -> /PA9
- J1 pad 29: unconnected-(J1-Pad29) -> GND
- J1 pad 3: unconnected-(J1-Pad3) -> /PG12
- J1 pad 30: unconnected-(J1-Pad30) -> GND
- J1 pad 31: unconnected-(J1-Pad31) -> /PJ12
- J1 pad 32: unconnected-(J1-Pad32) -> /PA8
- J1 pad 33: unconnected-(J1-Pad33) -> GND
- J1 pad 34: unconnected-(J1-Pad34) -> GND
- J1 pad 35: unconnected-(J1-Pad35) -> /PD3
- J1 pad 36: unconnected-(J1-Pad36) -> /PC8
- J1 pad 37: unconnected-(J1-Pad37) -> GND
- J1 pad 38: unconnected-(J1-Pad38) -> GND
- J1 pad 39: unconnected-(J1-Pad39) -> /PD4
- J1 pad 4: unconnected-(J1-Pad4) -> GND
- J1 pad 40: unconnected-(J1-Pad40) -> /PG7
- J1 pad 41: unconnected-(J1-Pad41) -> GND
- J1 pad 42: unconnected-(J1-Pad42) -> GND
- J1 pad 43: unconnected-(J1-Pad43) -> /PC12
- J1 pad 44: unconnected-(J1-Pad44) -> /PK0
- J1 pad 45: unconnected-(J1-Pad45) -> GND
- J1 pad 46: unconnected-(J1-Pad46) -> GND
- J1 pad 47: unconnected-(J1-Pad47) -> /PA15
- J1 pad 48: unconnected-(J1-Pad48) -> /PJ11
- J1 pad 49: unconnected-(J1-Pad49) -> GND
- J1 pad 5: unconnected-(J1-Pad5) -> GND
- J1 pad 50: unconnected-(J1-Pad50) -> GND
- J1 pad 51: unconnected-(J1-Pad51) -> /PA14
- J1 pad 52: unconnected-(J1-Pad52) -> /PB11
- J1 pad 53: unconnected-(J1-Pad53) -> GND
- J1 pad 54: unconnected-(J1-Pad54) -> GND
- J1 pad 55: unconnected-(J1-Pad55) -> /PC7
- J1 pad 56: unconnected-(J1-Pad56) -> /PJ8
- J1 pad 57: unconnected-(J1-Pad57) -> GND
- J1 pad 58: unconnected-(J1-Pad58) -> GND
- J1 pad 59: unconnected-(J1-Pad59) -> /PC6
- J1 pad 6: unconnected-(J1-Pad6) -> GND
- J1 pad 60: unconnected-(J1-Pad60) -> /PJ7
- J1 pad 61: unconnected-(J1-Pad61) -> GND
- J1 pad 62: unconnected-(J1-Pad62) -> GND
- J1 pad 63: unconnected-(J1-Pad63) -> /PK2
- J1 pad 64: unconnected-(J1-Pad64) -> /PB10
- J1 pad 65: unconnected-(J1-Pad65) -> GND
- J1 pad 66: unconnected-(J1-Pad66) -> GND
- J1 pad 67: unconnected-(J1-Pad67) -> /PG6
- J1 pad 68: unconnected-(J1-Pad68) -> /PJ5
- J1 pad 69: unconnected-(J1-Pad69) -> GND
- J1 pad 7: unconnected-(J1-Pad7) -> /PG10
- J1 pad 70: unconnected-(J1-Pad70) -> GND
- J1 pad 71: unconnected-(J1-Pad71) -> /PG3
- J1 pad 72: unconnected-(J1-Pad72) -> /PH7
- J1 pad 73: unconnected-(J1-Pad73) -> GND
- J1 pad 74: unconnected-(J1-Pad74) -> GND
- J1 pad 75: unconnected-(J1-Pad75) -> /PK1
- J1 pad 76: unconnected-(J1-Pad76) -> /PB13
- J1 pad 77: unconnected-(J1-Pad77) -> GND
- J1 pad 78: unconnected-(J1-Pad78) -> GND
- J1 pad 79: unconnected-(J1-Pad79) -> /PJ10
- J1 pad 8: unconnected-(J1-Pad8) -> GND
- J1 pad 80: unconnected-(J1-Pad80) -> /PB12
- J1 pad 81: unconnected-(J1-Pad81) -> GND
- J1 pad 82: unconnected-(J1-Pad82) -> GND
- J1 pad 83: unconnected-(J1-Pad83) -> /PJ9
- J1 pad 84: unconnected-(J1-Pad84) -> /PB14
- J1 pad 85: unconnected-(J1-Pad85) -> GND
- J1 pad 86: unconnected-(J1-Pad86) -> GND
- J1 pad 87: unconnected-(J1-Pad87) -> /PJ6
- J1 pad 88: unconnected-(J1-Pad88) -> /PB15
- J1 pad 89: unconnected-(J1-Pad89) -> GND
- J1 pad 9: unconnected-(J1-Pad9) -> GND
- J1 pad 90: unconnected-(J1-Pad90) -> GND
- J1 pad 91: unconnected-(J1-Pad91) -> /PD13
- J1 pad 92: unconnected-(J1-Pad92) -> /PD11
- J1 pad 93: unconnected-(J1-Pad93) -> GND
- J1 pad 94: unconnected-(J1-Pad94) -> GND
- J1 pad 95: unconnected-(J1-Pad95) -> /PD12
- J1 pad 96: unconnected-(J1-Pad96) -> /PH6
- J1 pad 97: unconnected-(J1-Pad97) -> GND
- J1 pad 98: unconnected-(J1-Pad98) -> GND
- J1 pad 99: unconnected-(J1-Pad99) -> GND
- J2 pad 10: unconnected-(J2-Pad10) -> GND
- J2 pad 100: unconnected-(J2-Pad100) -> GND
- J2 pad 11: unconnected-(J2-Pad11) -> GND
- J2 pad 14: unconnected-(J2-Pad14) -> GND
- J2 pad 15: unconnected-(J2-Pad15) -> GND
- J2 pad 16: unconnected-(J2-Pad16) -> GND
- J2 pad 17: unconnected-(J2-Pad17) -> /PA5
- J2 pad 18: unconnected-(J2-Pad18) -> GND
- J2 pad 19: unconnected-(J2-Pad19) -> /PA3
- J2 pad 2: unconnected-(J2-Pad2) -> GND
- J2 pad 20: unconnected-(J2-Pad20) -> GND
- J2 pad 21: unconnected-(J2-Pad21) -> /PA1_C
- J2 pad 22: unconnected-(J2-Pad22) -> GND
- J2 pad 23: unconnected-(J2-Pad23) -> GND
- J2 pad 25: unconnected-(J2-Pad25) -> /PA0_C
- J2 pad 27: unconnected-(J2-Pad27) -> /PA6
- J2 pad 29: unconnected-(J2-Pad29) -> /PC3_C
- J2 pad 3: unconnected-(J2-Pad3) -> GND
- J2 pad 31: unconnected-(J2-Pad31) -> /PC2_C
- J2 pad 33: unconnected-(J2-Pad33) -> /PH4
- J2 pad 35: unconnected-(J2-Pad35) -> /PA2
- J2 pad 37: unconnected-(J2-Pad37) -> GND
- J2 pad 39: unconnected-(J2-Pad39) -> +3V3
- J2 pad 41: unconnected-(J2-Pad41) -> +3V3
- J2 pad 43: unconnected-(J2-Pad43) -> +3V3
- J2 pad 44: unconnected-(J2-Pad44) -> GND
- J2 pad 45: unconnected-(J2-Pad45) -> +3V3
- J2 pad 46: unconnected-(J2-Pad46) -> GND
- J2 pad 47: unconnected-(J2-Pad47) -> +3V3
- J2 pad 48: unconnected-(J2-Pad48) -> GND
- J2 pad 49: unconnected-(J2-Pad49) -> +3V3
- J2 pad 51: unconnected-(J2-Pad51) -> GND
- J2 pad 53: unconnected-(J2-Pad53) -> GND
- J2 pad 57: unconnected-(J2-Pad57) -> /PC13
- J2 pad 59: unconnected-(J2-Pad59) -> /PE5
- J2 pad 6: unconnected-(J2-Pad6) -> GND
- J2 pad 61: unconnected-(J2-Pad61) -> /PE4
- J2 pad 63: unconnected-(J2-Pad63) -> /PE3
- J2 pad 65: unconnected-(J2-Pad65) -> /PB7
- J2 pad 67: unconnected-(J2-Pad67) -> /PB6
- J2 pad 69: unconnected-(J2-Pad69) -> /PB5
- J2 pad 7: unconnected-(J2-Pad7) -> GND
- J2 pad 71: unconnected-(J2-Pad71) -> /PK3
- J2 pad 73: unconnected-(J2-Pad73) -> GND
- J2 pad 75: unconnected-(J2-Pad75) -> /PK4
- J2 pad 77: unconnected-(J2-Pad77) -> GND
- J2 pad 79: unconnected-(J2-Pad79) -> /PK5
- J2 pad 8: /PC4 -> GND
- J2 pad 81: unconnected-(J2-Pad81) -> GND
- J2 pad 83: unconnected-(J2-Pad83) -> /PG13
- J2 pad 85: unconnected-(J2-Pad85) -> GND
- J2 pad 87: unconnected-(J2-Pad87) -> GND
- J2 pad 89: unconnected-(J2-Pad89) -> GND
- J2 pad 91: unconnected-(J2-Pad91) -> GND
- J2 pad 97: /ex_VBAT -> GND
- J2 pad 98: /ex_VBAT -> GND
- J2 pad 99: unconnected-(J2-Pad99) -> GND
- U1 pad A8: /mcu/PK5 -> /PK5
- U1 pad A9: /mcu/PG10 -> /PG10
- U1 pad B10: /mcu/PJ15 -> /PJ15
- U1 pad B8: /mcu/PK4 -> /PK4
- U1 pad B9: /mcu/PG11 -> /PG11
- U1 pad C8: /mcu/PK3 -> /PK3
- U1 pad C9: /mcu/PG12 -> /PG12
- U1 pad D11: /mcu/PJ12 -> /PJ12
- U1 pad D9: /mcu/PG13 -> /PG13
- U1 pad F16: /mcu/PG7 -> /PG7
- U1 pad G15: /mcu/PG6 -> /PG6
- U1 pad H15: /mcu/PG3 -> /PG3
- U1 pad H17: /mcu/PK2 -> /PK2
- U1 pad J14: /mcu/PK0 -> /PK0
- U1 pad J15: /mcu/PK1 -> /PK1
- U1 pad K14: /mcu/PJ11 -> /PJ11
- U1 pad L14: /mcu/PJ10 -> /PJ10
- U1 pad M14: /mcu/PJ9 -> /PJ9
- U1 pad N13: /mcu/PJ8 -> /PJ8
- U1 pad N14: /mcu/PJ7 -> /PJ7
- U1 pad N15: /mcu/PJ6 -> /PJ6
- U1 pad P3: /mcu/PH4 -> /PH4
- U1 pad R12: /mcu/PJ5 -> /PJ5
- U1 pad T11: /mcu/PH6 -> /PH6
- U1 pad T4: /PC4 -> GND
- U1 pad U13: /mcu/PH7 -> /PH7
Routing:
- net GND: track 82.4 -> 115.1 mm, vias 64 -> 67
- net /PG13: track 0.00 -> 28.8 mm, vias 0 -> 1
- net /PK3: track 0.00 -> 28.5 mm, vias 0 -> 1
- net /PK4: track 0.00 -> 27.4 mm, vias 0 -> 1
- net /PK5: track 0.00 -> 26.4 mm, vias 0 -> 1
- net /PJ12: track 0.00 -> 24.3 mm, vias 0 -> 1
- net /PG12: track 0.00 -> 23.9 mm, vias 0 -> 1
- net /PJ15: track 0.00 -> 23.5 mm, vias 0 -> 1
- net /PG11: track 0.00 -> 23.4 mm, vias 0 -> 1
- net /PG10: track 0.00 -> 22.4 mm, vias 0 -> 1
- net /PB5: track 1.60 -> 23.3 mm, vias 0 -> 1
- net /PB7: track 3.40 -> 24.5 mm, vias 0 -> 1
- net /PC12: track 3.85 -> 23.9 mm, vias 0 -> 1
- net /PD4: track 2.20 -> 22.0 mm, vias 0 -> 1
- net /PD3: track 3.17 -> 22.8 mm, vias 0 -> 1
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Other:
- outline, holes or cut-outs redrawn
- board text added: "H750core v0.1"
- board text added: "LDO"
- board text added: "Pegnitz digital."
- board text added: "VCAP"
- board text added: "VREF"
